Commit message: urdf, xacro file fix
lidar sensor joint turn for 180 degree

File: urdf/zzangdol_ai_car.urdf (robot description, URDF)
Before this commit: robot zzangdol_ai_car, 8 links, 7 joints
Joints:
- joint lidar_joint: origin xyz=0.15 0 0.1 rpy=0 0 0 -> xyz=0.15 0 0.1 rpy=0 0 3.141592653589793

File: urdf/zzangdol_ai_car.urdf.xacro (robot description, xacro)
@@ -121,5 +121,5 @@
   </link>
   <joint name="lidar_joint" type="fixed">
-    <origin xyz="0.15 0 0.1" rpy="0 0 0"/>
+    <origin xyz="0.15 0 0.1" rpy="0 0 ${M_PI}"/>
     <parent link="base_link"/>
     <child link="lidar_link"/>
